File: packages/eda/eda.kicad_pcb (KiCad board)
At the start: 2 copper layers, 19 parts, among them U1 Pico

Commit message: chore: minor changes
Parts:
- moved LCD1 6.28 mm to (147.5, 84.5)
Routing:
- net /Buzzer: track 16.4 -> 0.00 mm
- net /LCD_RST: track 17.5 -> 8.49 mm
- net /LCD_RS: track 17.0 -> 8.71 mm
- net /LCD_SDA: track 16.6 -> 8.93 mm
- net /LCD_CS: track 14.9 -> 7.23 mm
- net /LCD_CLK: track 15.8 -> 9.16 mm
- net /5V: track 192.6 -> 198.8 mm
- net /GND: track 215.9 -> 219.7 mm
- net /3.3V: track 152.7 -> 154.2 mm

Commit message: chore: minor changes
Parts:
- moved SwitchConfig1 11.5 mm to (127.0, 81.5), turned to 180 degrees
- moved StepperDiscard1 3.78 mm to (140.7, 120.6)
- moved MotorDiscard1 3.74 mm to (140.8, 133.1)
- moved SensorCheck1 3.74 mm to (158.3, 126.2)
- moved SensorDrop1 3.74 mm to (153.3, 126.2)
- moved SwitchPower1 2.11 mm to (166.5, 130.5)
- moved Buzzer1 0.65 mm to (147.5, 75.0)
Routing:
- net /Buzzer: track 0.00 -> 15.9 mm
- net /3.3V: track 154.2 -> 147.3 mm
- net /5V: track 198.8 -> 193.4 mm
- net /SW: track 5.42 -> 10.4 mm
- net /GND: track 219.7 -> 215.2 mm
- net /Serv10: track 22.6 -> 18.6 mm
- net /Serv01: track 23.1 -> 19.2 mm
- net /SDC: track 11.7 -> 14.7 mm
- net /Serv11: track 19.5 -> 16.8 mm
- net /GNDP: track 17.6 -> 20.0 mm
- net /StD23: track 11.2 -> 12.9 mm
- net /StD24: track 11.2 -> 12.8 mm
- net /StD22: track 12.1 -> 13.7 mm
- net /StD21: track 12.1 -> 13.7 mm
- net /SDD: track 12.7 -> 12.0 mm

Commit message: chore: minor changes
Parts:
- added ButtonLink1: ~, Connector_PinHeader_2.54mm:PinHeader_1x02_P2.54mm_Vertical, F.Cu at (149.5, 118.5)
- added R1: 330, Resistor_THT:R_Axial_DIN0207_L6.3mm_D2.5mm_P7.62mm_Horizontal, F.Cu at (190.0, 76.2)
- added R10: 220, Resistor_THT:R_Axial_DIN0207_L6.3mm_D2.5mm_P7.62mm_Horizontal, F.Cu at (124.0, 76.2)
- added R11: 220, Resistor_THT:R_Axial_DIN0207_L6.3mm_D2.5mm_P7.62mm_Horizontal, F.Cu at (140.2, 117.3)
- added R12: 220, Resistor_THT:R_Axial_DIN0207_L6.3mm_D2.5mm_P7.62mm_Horizontal, F.Cu at (135.7, 117.3)
- added R13: 220, Resistor_THT:R_Axial_DIN0207_L6.3mm_D2.5mm_P7.62mm_Horizontal, F.Cu at (131.2, 117.3)
- added R14: 220, Resistor_THT:R_Axial_DIN0207_L6.3mm_D2.5mm_P7.62mm_Horizontal, F.Cu at (126.7, 117.3)
- added R15: 220, Resistor_THT:R_Axial_DIN0207_L6.3mm_D2.5mm_P7.62mm_Horizontal, F.Cu at (152.5, 83.8)
- added R16: 220, Resistor_THT:R_Axial_DIN0207_L6.3mm_D2.5mm_P7.62mm_Horizontal, F.Cu at (157.0, 83.8)
- added R17: 220, Resistor_THT:R_Axial_DIN0207_L6.3mm_D2.5mm_P7.62mm_Horizontal, F.Cu at (161.5, 83.8)
- added R18: 220, Resistor_THT:R_Axial_DIN0207_L6.3mm_D2.5mm_P7.62mm_Horizontal, F.Cu at (166.0, 83.8)
- added R2: 330, Resistor_THT:R_Axial_DIN0207_L6.3mm_D2.5mm_P7.62mm_Horizontal, F.Cu at (185.0, 76.2)
- added R3: 330, Resistor_THT:R_Axial_DIN0207_L6.3mm_D2.5mm_P7.62mm_Horizontal, F.Cu at (180.0, 76.2)
- added R4: 330, Resistor_THT:R_Axial_DIN0207_L6.3mm_D2.5mm_P7.62mm_Horizontal, F.Cu at (175.0, 76.2)
- added R5: 330, Resistor_THT:R_Axial_DIN0207_L6.3mm_D2.5mm_P7.62mm_Horizontal, F.Cu at (145.0, 124.9)
- added R6: 330, Resistor_THT:R_Axial_DIN0207_L6.3mm_D2.5mm_P7.62mm_Horizontal, F.Cu at (142.0, 76.2)
- added R7: 330, Resistor_THT:R_Axial_DIN0207_L6.3mm_D2.5mm_P7.62mm_Horizontal, F.Cu at (137.5, 76.2)
- added R8: 330, Resistor_THT:R_Axial_DIN0207_L6.3mm_D2.5mm_P7.62mm_Horizontal, F.Cu at (133.0, 76.2)
- added R9: 330, Resistor_THT:R_Axial_DIN0207_L6.3mm_D2.5mm_P7.62mm_Horizontal, F.Cu at (128.5, 76.2)
- SwitchConfig1, SwitchPower1: footprint Connector_PinHeader_2.00mm:PinHeader_1x02_P2.00mm_Vertical -> Connector_PinHeader_2.54mm:PinHeader_1x02_P2.54mm_Vertical
- moved Buzzer1 54.6 mm to (145.0, 129.5), turned to 90 degrees
- moved LCD1 12.9 mm to (147.0, 71.6)
- moved SwitchConfig1 11.4 mm to (121.5, 71.5), turned to 90 degrees
- moved MotorDiscard1 8.93 mm to (140.0, 142.0)
- moved StepperDiscard1 8.92 mm to (140.0, 129.5)
- moved StepperDrawer1 8.31 mm to (152.8, 71.6)
- moved MotorDrawer1 8.04 mm to (153.0, 59.6)
- moved Servo0-0 7.61 mm to (190.1, 66.4)
- moved Servo0-1 7.61 mm to (185.1, 66.4)
- moved Servo1-0 7.61 mm to (180.1, 66.4)
- moved Servo1-1 7.61 mm to (175.1, 66.4)
- moved SwitchPower1 4.37 mm to (168.0, 134.6)
- moved Diode1 4.23 mm to (172.6, 124.5)
- moved Diode2 4.23 mm to (181.6, 124.5)
- moved PowerMCU1 4.23 mm to (177.1, 132.1)
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Connections:
- net /SDC renamed /SC
- net /SDD renamed /SD
- Buzzer1 pad 2: /Buzzer -> Net-(Buzzer1-Pin_2)
- LCD1 pad 10: /LCD_CS -> Net-(LCD1-Pin_10)
- LCD1 pad 6: /LCD_CLK -> Net-(LCD1-Pin_6)
- LCD1 pad 7: /LCD_SDA -> Net-(LCD1-Pin_7)
- LCD1 pad 8: /LCD_RS -> Net-(LCD1-Pin_8)
- LCD1 pad 9: /LCD_RST -> Net-(LCD1-Pin_9)
- Servo0-0 pad 3: /Serv00 -> Net-(Servo0-0-Pin_3)
- Servo0-1 pad 3: /Serv01 -> Net-(Servo0-1-Pin_3)
- Servo1-0 pad 3: /Serv10 -> Net-(Servo1-0-Pin_3)
- Servo1-1 pad 3: /Serv11 -> Net-(Servo1-1-Pin_3)
- StepperDiscard1 pad 1: /StD24 -> Net-(StepperDiscard1-I1)
- StepperDiscard1 pad 2: /StD23 -> Net-(StepperDiscard1-I2)
- StepperDiscard1 pad 3: /StD22 -> Net-(StepperDiscard1-I3)
- StepperDiscard1 pad 4: /StD21 -> Net-(StepperDiscard1-I4)
- StepperDrawer1 pad 1: /StD14 -> Net-(StepperDrawer1-I1)
- StepperDrawer1 pad 2: /StD13 -> Net-(StepperDrawer1-I2)
- StepperDrawer1 pad 3: /StD12 -> Net-(StepperDrawer1-I3)
- StepperDrawer1 pad 4: /StD11 -> Net-(StepperDrawer1-I4)
- U1 pad 12: /Buzzer -> unconnected-(U1-GPIO9-Pad12)
- U1 pad 26: unconnected-(U1-GPIO20-Pad26) -> /Buzzer
- U1 pad 27: unconnected-(U1-GPIO21-Pad27) -> /BTN
Routing:
- net /GND: track 215.2 -> 262.8 mm
- net /5V: track 193.4 -> 212.4 mm
- net /SW: track 10.4 -> 24.4 mm
- net /BTN: track 0.00 -> 12.0 mm
- net Net-(StepperDrawer1-I4): track 0.00 -> 7.86 mm
- net Net-(StepperDiscard1-I4): track 0.00 -> 7.83 mm
- net /3.3V: track 147.3 -> 139.5 mm
- net Net-(LCD1-Pin_6): track 0.00 -> 7.62 mm
- net Net-(LCD1-Pin_10): track 0.00 -> 7.62 mm
- net Net-(Buzzer1-Pin_2): track 0.00 -> 6.44 mm
- net Net-(StepperDrawer1-I3): track 0.00 -> 6.16 mm
- net Net-(StepperDiscard1-I3): track 0.00 -> 6.15 mm
- net /Buzzer: track 15.9 -> 10.0 mm
- net Net-(LCD1-Pin_7): track 0.00 -> 5.79 mm
- net /StD21: track 13.7 -> 7.93 mm
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