File: packages/eda/eda.kicad_pcb (KiCad board)
At the start: 2 copper layers, 38 parts, among them U1 Pico

Commit message: fix(eda): vcc
Parts:
- MotorDiscard1, MotorDrawer1: footprint Connector_PinHeader_2.00mm:PinHeader_1x04_P2.00mm_Vertical -> Connector_PinHeader_2.54mm:PinHeader_1x05_P2.54mm_Vertical
- moved MotorDiscard1 10.4 mm to (129.8, 144.1), turned to 90 degrees
- moved MotorDrawer1 10.2 mm to (163.1, 57.8), turned to -90 degrees
- moved SwitchPower1 2.53 mm to (168.0, 132.1), turned to 0 degrees
Connections:
- MotorDiscard1 pad 1: Net-(MotorDiscard1-Pin_1) -> /5V
- MotorDrawer1 pad 1: Net-(MotorDrawer1-Pin_1) -> /5V
- StepperDiscard1 pad 13: Net-(MotorDiscard1-Pin_4) -> Net-(MotorDiscard1-Pin_2)
- StepperDiscard1 pad 15: Net-(MotorDiscard1-Pin_2) -> Net-(MotorDiscard1-Pin_4)
- StepperDiscard1 pad 16: Net-(MotorDiscard1-Pin_1) -> Net-(MotorDiscard1-Pin_5)
- StepperDrawer1 pad 13: Net-(MotorDrawer1-Pin_4) -> Net-(MotorDrawer1-Pin_2)
- StepperDrawer1 pad 15: Net-(MotorDrawer1-Pin_2) -> Net-(MotorDrawer1-Pin_4)
- StepperDrawer1 pad 16: Net-(MotorDrawer1-Pin_1) -> Net-(MotorDrawer1-Pin_5)
- SwitchPower1 pad 1: /GNDP -> /GND
- SwitchPower1 pad 2: /GND -> /GNDP
Routing:
- net /5V: track 212.4 -> 238.7 mm
- net Net-(MotorDiscard1-Pin_5): track 0.00 -> 7.06 mm
- net Net-(MotorDrawer1-Pin_5): track 0.00 -> 6.54 mm
- net Net-(MotorDiscard1-Pin_1): track 4.91 -> 0.00 mm
- net Net-(MotorDrawer1-Pin_1): track 4.46 -> 0.00 mm
- net /GND: track 263.0 -> 267.1 mm
- net Net-(MotorDiscard1-Pin_2): track 5.07 -> 7.06 mm
- net Net-(MotorDiscard1-Pin_3): track 5.29 -> 7.06 mm
- net Net-(MotorDrawer1-Pin_2): track 4.52 -> 6.26 mm
- net Net-(MotorDrawer1-Pin_3): track 4.74 -> 6.26 mm
- net Net-(MotorDiscard1-Pin_4): track 5.55 -> 7.06 mm
- net Net-(MotorDrawer1-Pin_4): track 4.97 -> 6.26 mm

Commit message: chore: minor changes
Parts:
- LCD1: footprint Connector_PinHeader_2.00mm:PinHeader_1x10_P2.00mm_Vertical -> Connector_PinHeader_2.54mm:PinHeader_1x10_P2.54mm_Vertical
- moved SwitchConfig1 2.46 mm to (119.0, 71.6), turned to 0 degrees
- moved MotorDrawer1 0.38 mm to (162.7, 57.8)
- moved StepperDrawer1 0.27 mm to (152.5, 71.6)
- moved LCD1 0.06 mm to (146.9, 71.6)
Connections:
- SwitchConfig1 pad 1: /SW -> /GND
- SwitchConfig1 pad 2: /GND -> /SW
Routing:
- net Net-(LCD1-Pin_10): track 7.62 -> 4.60 mm
- net Net-(LCD1-Pin_8): track 4.57 -> 7.08 mm
- net /GND: track 267.1 -> 269.5 mm
- net Net-(LCD1-Pin_6): track 7.62 -> 9.86 mm
- net Net-(LCD1-Pin_7): track 5.79 -> 7.95 mm
- net Net-(StepperDrawer1-I3): track 6.16 -> 7.21 mm

Commit message: chore: minor changes
Routing:
- net Net-(StepperDiscard1-I3): track 6.15 -> 7.12 mm
Changed lines of the file:
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@@
 	(segment
 		(start 134.96 129.5)
-		(end 134.96 128.74)
+		(end 134.96 127.086)
 		(width 0.8)
 		(layer "B.Cu")
@@
 	)
 	(segment
-		(start 134.96 128.74)
+		(start 134.96 127.086)
+		(end 132.804 124.93)
+		(width 0.8)
+		(layer "B.Cu")
+		(net "Net-(StepperDiscard1-I3)")
+	)
+	(segment
+		(start 132.804 124.93)
 		(end 131.15 124.93)
 		(width 0.8)
@@
 	)
 	(segment
-		(start 132.42 129.211572)
-		(end 128.138428 124.93)
-		(width 0.8)
-		(layer "B.Cu")
-		(net "Net-(StepperDiscard1-I4)")
-	)
-	(segment
-		(start 128.138428 124.93)
+		(start 128.232 124.93)
 		(end 126.65 124.93)
 		(width 0.8)
@@
 	(segment
 		(start 132.42 129.5)
-		(end 132.42 129.211572)
+		(end 132.42 129.118)
 		(width 0.8)
 		(layer "B.Cu")
+		(net "Net-(StepperDiscard1-I4)")
+	)
+	(segment
+		(start 132.42 129.118)
+		(end 128.232 124.93)
+		(width 0.8)
+		(layer "B.Cu")

Commit message: chore: bump deps
Parts:
- added Fan1: ~, Connector_PinHeader_2.54mm:PinHeader_1x02_P2.54mm_Vertical, F.Cu at (152.9, 134.3)
- added Fan2: ~, Connector_PinHeader_2.54mm:PinHeader_1x02_P2.54mm_Vertical, F.Cu at (152.9, 144.1)
- added R19: 330, Resistor_SMD:R_1206_3216Metric_Pad1.30x1.75mm_HandSolder, F.Cu at (128.7, 121.2)
- PowerMCU1, PowerPer1: footprint Connector_PinHeader_2.54mm:PinHeader_1x02_P2.54mm_Vertical -> Connector_Samtec_HPM_THT:Samtec_HPM-02-01-x-S_Straight_1x02_Pitch5.08mm
- R1, R10, R11, R12, R13, R14, R15, R16, R17, R18, R2, R3, R4, R5, R6, R7, R8, R9: footprint Resistor_THT:R_Axial_DIN0207_L6.3mm_D2.5mm_P7.62mm_Horizontal -> Resistor_SMD:R_1206_3216Metric_Pad1.30x1.75mm_HandSolder
- moved Servo1-0 80.9 mm to (203.0, 144.1), turned to -90 degrees
- moved MotorDiscard1 78.2 mm to (117.0, 67.0), turned to 0 degrees
- moved Servo0-1 77.8 mm to (190.4, 144.1), turned to -90 degrees
- moved SwitchConfig1 74.8 mm to (159.7, 134.3), turned to 90 degrees
- moved Servo1-1 73.7 mm to (203.0, 134.6), turned to -90 degrees
- moved R10 71.1 mm to (195.1, 74.7), turned to 180 degrees
- moved PowerPer1 70.1 mm to (117.0, 144.0), turned to 90 degrees
- moved Servo0-0 68.2 mm to (190.4, 134.6), turned to -90 degrees
- moved R9 66.6 mm to (195.1, 77.7), turned to 180 degrees
- moved Diode2 66.2 mm to (116.3, 135.8), turned to 0 degrees
- moved R8 62.2 mm to (195.1, 80.8), turned to 180 degrees
- moved LCD1 61.9 mm to (203.1, 97.8), turned to 180 degrees
- moved R7 58.1 mm to (195.1, 83.8), turned to 180 degrees
- moved R4 57.1 mm to (200.2, 127.4), turned to 90 degrees
- moved MotorDrawer1 56.8 mm to (117.0, 91.6), turned to 0 degrees
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Connections:
- ButtonLink1 pad 1: /BTN -> Net-(ButtonLink1-Pin_1)
Routing:
- net /StD11: track 9.36 -> 120.1 mm, vias 0 -> 1
- net /StD12: track 8.55 -> 116.9 mm, vias 0 -> 1
- net /StD13: track 9.17 -> 109.7 mm, vias 0 -> 1
- net /StD14: track 8.36 -> 106.6 mm, vias 0 -> 1
- net /SW: track 23.9 -> 70.5 mm
- net /BTN: track 12.0 -> 57.1 mm
- net /Buzzer: track 10.0 -> 48.5 mm
- net /VCC: track 15.1 -> 51.6 mm
- net /GNDP: track 18.2 -> 49.2 mm
- net Net-(Servo0-1-Pin_3): track 4.62 -> 27.3 mm
- net /SC: track 10.9 -> 29.8 mm
- net /Serv11: track 15.1 -> 31.2 mm
- net /3.3V: track 139.9 -> 155.8 mm
- net /SD: track 9.89 -> 23.9 mm
- net /GND: track 269.5 -> 283.4 mm
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Other:
- board outline added: 100 x 100 mm
- board text added: "22653991 - Tran Tien 22637811 - Dao Anh Huy"

Commit message: chore: minor changes
Parts:
- moved LCD1 0.51 mm to (203.1, 97.3)
- moved R10 0.25 mm to (195.1, 74.4)
- moved R6 0.25 mm to (195.1, 87.2)
- moved R9 0.25 mm to (195.1, 77.4)
- moved R7 0.25 mm to (195.1, 83.5)
- moved R8 0.25 mm to (195.1, 80.6)
Routing:
- net /3.3V: track 155.8 -> 282.6 mm
- net /GND: track 283.4 -> 295.1 mm
- net /SW: track 70.5 -> 77.6 mm
- net Net-(Servo0-1-Pin_3): track 27.3 -> 20.2 mm
- net /5V: track 226.5 -> 221.1 mm
- net /BTN: track 57.1 -> 52.6 mm
- net /Serv10: track 26.7 -> 22.4 mm
- net /Serv11: track 31.2 -> 27.3 mm
- net Net-(MotorDrawer1-Pin_4): track 12.1 -> 9.97 mm
- net /Serv01: track 18.6 -> 16.5 mm
- net /Buzzer: track 48.5 -> 46.7 mm
- net /SD: track 23.9 -> 22.4 mm
- net Net-(Buzzer1-Pin_2): track 9.66 -> 11.1 mm
- net Net-(Diode1-A): track 11.2 -> 12.5 mm
- net /StD14: track 106.6 -> 107.9 mm
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- added copper zone on F.Cu, net (none)
- added copper zone on B.Cu, net /GND
- added copper zone on F.Cu, net /GND
