File: packages/eda/eda.kicad_sch (KiCad schematic)
At the start: 19 parts, among them U1 Pico

Commit message: chore: minor changes
Parts:
- added ButtonLink1: (no value), Connector_PinHeader_2.54mm:PinHeader_1x02_P2.54mm_Vertical, symbol Connector:Conn_01x02_Pin
- added R1, R2, R3, R4, R5, R6, R7, R8, R9: 330, Resistor_THT:R_Axial_DIN0207_L6.3mm_D2.5mm_P7.62mm_Horizontal, symbol Device:R
- added R10, R11, R12, R13, R14, R15, R16, R17, R18: 220, Resistor_THT:R_Axial_DIN0207_L6.3mm_D2.5mm_P7.62mm_Horizontal, symbol Device:R
- SwitchConfig1, SwitchPower1: footprint Connector_PinHeader_2.00mm:PinHeader_1x02_P2.00mm_Vertical -> Connector_PinHeader_2.54mm:PinHeader_1x02_P2.54mm_Vertical
Connections:
- net Buzzer: now also U1.26 (GPIO20), R5.2; no longer Buzzer1.2 (Pin_2), U1.12 (GPIO9)
- net GND: now also ButtonLink1.2 (Pin_2)
- net LCD_CLK: now also R6.2; no longer LCD1.6 (Pin_6)
- net LCD_CS: now also R10.2; no longer LCD1.10 (Pin_10)
- net LCD_RS: now also R8.2; no longer LCD1.8 (Pin_8)
- net LCD_RST: now also R9.2; no longer LCD1.9 (Pin_9)
- net LCD_SDA: now also R7.2; no longer LCD1.7 (Pin_7)
- net Serv00: now also R1.2; no longer Servo0-0.3 (Pin_3)
- net Serv01: now also R2.2; no longer Servo0-1.3 (Pin_3)
- net Serv10: now also R3.2; no longer Servo1-0.3 (Pin_3)
- net Serv11: now also R4.2; no longer Servo1-1.3 (Pin_3)
- net StD11: now also R18.1; no longer StepperDrawer1.4 (I4)
- net StD12: now also R17.1; no longer StepperDrawer1.3 (I3)
- net StD13: now also R16.1; no longer StepperDrawer1.2 (I2)
- net StD14: now also R15.1; no longer StepperDrawer1.1 (I1)
- net StD21: now also R14.1; no longer StepperDiscard1.4 (I4)
- net StD22: now also R13.1; no longer StepperDiscard1.3 (I3)
- net StD23: now also R12.1; no longer StepperDiscard1.2 (I2)
- net StD24: now also R11.1; no longer StepperDiscard1.1 (I1)
- net BTN: now reaches U1.27 (GPIO21)
- net BTN: now also ButtonLink1.1 (Pin_1)
- net SDC renamed SC
- net SDD renamed SD
- new net: R14.2, StepperDiscard1.4 (I4)
- new net: R4.1, Servo1-1.3 (Pin_3)
- new net: R18.2, StepperDrawer1.4 (I4)
- new net: Buzzer1.2 (Pin_2), R5.1
- new net: R17.2, StepperDrawer1.3 (I3)
- new net: R3.1, Servo1-0.3 (Pin_3)
- new net: R1.1, Servo0-0.3 (Pin_3)
- new net: R16.2, StepperDrawer1.2 (I2)
- new net: R11.2, StepperDiscard1.1 (I1)
- new net: R12.2, StepperDiscard1.2 (I2)
- new net: R13.2, StepperDiscard1.3 (I3)
- new net: LCD1.8 (Pin_8), R8.1
- new net: R15.2, StepperDrawer1.1 (I1)
- new net: LCD1.10 (Pin_10), R10.1
- new net: LCD1.7 (Pin_7), R7.1
- new net: R2.1, Servo0-1.3 (Pin_3)
- new net: LCD1.6 (Pin_6), R6.1
- new net: LCD1.9 (Pin_9), R9.1
Other:
- moved on the sheet: Buzzer1, LCD1, MotorDiscard1, MotorDrawer1, SensorCheck1, SensorDrop1, Servo0-0, Servo0-1, Servo1-0, Servo1-1, StepperDiscard1, StepperDrawer1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

Commit message: fix(eda): vcc
Parts:
- removed MotorDiscard1, MotorDrawer1: (no value), Connector_PinHeader_2.00mm:PinHeader_1x04_P2.00mm_Vertical, symbol Connector:Conn_01x04_Pin
- added MotorDiscard1, MotorDrawer1: (no value), Connector_PinHeader_2.54mm:PinHeader_1x05_P2.54mm_Vertical, symbol Connector:Conn_01x05_Pin
Connections:
- net 5V: now also MotorDiscard1.1 (Pin_1), MotorDrawer1.1 (Pin_1)
- net GND: now also SwitchPower1.1 (Pin_1); no longer SwitchPower1.2 (Pin_2)
- net GNDP: now also SwitchPower1.2 (Pin_2); no longer SwitchPower1.1 (Pin_1)
- net at StepperDiscard1.13 (O4): now also MotorDiscard1.2 (Pin_2)
- net at StepperDiscard1.14 (O3): now also MotorDiscard1.3 (Pin_3)
- net at StepperDiscard1.15 (O2): now also MotorDiscard1.4 (Pin_4)
- net at StepperDiscard1.16 (O1): now also MotorDiscard1.5 (Pin_5)
- net at StepperDrawer1.16 (O1): now also MotorDrawer1.5 (Pin_5)
- net at StepperDrawer1.15 (O2): now also MotorDrawer1.4 (Pin_4)
- net at StepperDrawer1.14 (O3): now also MotorDrawer1.3 (Pin_3)
- net at StepperDrawer1.13 (O4): now also MotorDrawer1.2 (Pin_2)
Changed lines of the file:
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@@
 	(wire
 		(pts
-			(xy 113.03 111.76) (xy 128.27 111.76)
-		)
-		(stroke
-			(width 0)
-			(type default)
-		)
-	)
-	(wire
-		(pts
 			(xy 120.65 91.44) (xy 128.27 91.44)
 		)
@@
 	(wire
 		(pts
+			(xy 113.03 111.76) (xy 128.27 111.76)
+		)
+		(stroke
+			(width 0)
+			(type default)
+		)
+	)
+	(wire
+		(pts
 			(xy 133.35 102.87) (xy 138.43 102.87)
 		)
@@
 	(wire
 		(pts
+			(xy 167.64 147.32) (xy 172.72 147.32)
+		)
+		(stroke
+			(width 0)
+			(type default)
+		)
+	)
+	(wire
+		(pts
+			(xy 167.64 113.03) (xy 171.45 113.03)
+		)
+		(stroke
+			(width 0)
+			(type default)
+		)
+	)
+	(wire
+		(pts
 			(xy 128.27 39.37) (xy 113.03 39.37)
 		)
@@
 		)
 	)
+	(label "5V"
+		(at 167.64 113.03 0)
+		(effects
+			(font
+				(size 1.27 1.27)
+			)
+			(justify left bottom)
+		)
+	)
 	(label "GND"
 		(at 177.8 123.19 180)
@@
 		)
 	)
+	(label "5V"
+		(at 167.64 147.32 0)
+		(effects
+			(font
+				(size 1.27 1.27)
+			)
+			(justify left bottom)
+		)
+	)
 	(label "Serv00"
 		(at 133.35 35.56 0)
@@
 	(symbol
 		(lib_id "Connector:Conn_01x02_Pin")
-		(at 107.95 111.76 0)
+		(at 107.95 114.3 0)
+		(mirror x)
 		(unit 1)
 		(body_style 1)
@@
 		(in_pos_files yes)
 		(dnp no)
-		(fields_autoplaced yes)
 		(property "Reference" "SwitchPower1"
-			(at 108.585 109.22 0)
+			(at 107.95 109.22 0)
 			(show_name no)
 			(do_not_autoplace no)
@@
 		)
 		(property "Value" ""
-			(at 108.585 109.22 0)
+			(at 108.585 116.84 0)
 			(show_name no)
 			(do_not_autoplace no)
@@
 		)
 		(property "Footprint" "Connector_PinHeader_2.54mm:PinHeader_1x02_P2.54mm_Vertical"
-			(at 107.95 111.76 0)
+			(at 107.95 114.3 0)
 			(hide yes)
 			(show_name no)
@@
 		)
 		(property "Datasheet" ""
-			(at 107.95 111.76 0)
+			(at 107.95 114.3 0)
 			(hide yes)
 			(show_name no)
@@
 		)
 		(property "Description" "Generic connector, single row, 01x02, script generated"
-			(at 107.95 111.76 0)
+			(at 107.95 114.3 0)
 			(hide yes)
 			(show_name no)
@@
 	)
 	(symbol
-		(lib_id "Connector:Conn_01x04_Pin")
-		(at 176.53 105.41 0)
-		(mirror y)
-		(unit 1)
-		(body_style 1)
-		(exclude_from_sim no)
-		(in_bom yes)
-		(on_board yes)
-		(in_pos_files yes)
-		(dnp no)
-		(property "Reference" "MotorDrawer1"
-			(at 176.53 100.33 0)
-			(show_name no)
-			(do_not_autoplace no)
-			(effects
-				(font
-					(size 1.27 1.27)
-				)
-				(justify left)
-			)
-		)
-		(property "Value" ""
-			(at 175.895 100.33 0)
-			(show_name no)
-			(do_not_autoplace no)
-			(effects
-				(font
-					(size 1.27 1.27)
-				)
-			)
-		)
-		(property "Footprint" "Connector_PinHeader_2.00mm:PinHeader_1x04_P2.00mm_Vertical"
-			(at 176.53 105.41 0)
-			(hide yes)
-			(show_name no)
-			(do_not_autoplace no)
-			(effects
-				(font
-					(size 1.27 1.27)
-				)
-			)
-		)
-		(property "Datasheet" ""
-			(at 176.53 105.41 0)
-			(hide yes)
-			(show_name no)
-			(do_not_autoplace no)
-			(effects
-				(font
-					(size 1.27 1.27)
-				)
-			)
-		)
-		(property "Description" "Generic connector, single row, 01x04, script generated"
-			(at 176.53 105.41 0)
-			(hide yes)
-			(show_name no)
-			(do_not_autoplace no)
-			(effects
-				(font
-					(size 1.27 1.27)
-				)
-			)
-		)
-		(pin "4"
-		)
-		(pin "1"
-		)
-		(pin "2"
-		)
-		(pin "3"
-		)
-		(instances
-			(project "eda"
-				(path "/42a0047f-f4da-41b6-a5bf-510bae675ffb"
-					(reference "MotorDrawer1")
-					(unit 1)
-				)
-			)
-		)
-	)
-	(symbol
 		(lib_id "Device:R")
 		(at 142.24 102.87 90)
@@
 	)
 	(symbol
+		(lib_id "Connector:Conn_01x05_Pin")
+		(at 176.53 107.95 180)
+		(unit 1)
+		(body_style 1)
+		(exclude_from_sim no)
+		(in_bom yes)
+		(on_board yes)
+		(in_pos_files yes)
+		(dnp no)
+		(property "Reference" "MotorDrawer1"
+			(at 176.53 100.33 0)
+			(show_name no)
+			(do_not_autoplace no)
+			(effects
+				(font
+					(size 1.27 1.27)
+				)
+				(justify left)
+			)
+		)
+		(property "Value" ""
+			(at 177.8 106.6801 0)
+			(show_name no)
+			(do_not_autoplace no)
+			(effects
+				(font
+					(size 1.27 1.27)
+				)
+				(justify right)
+			)
+		)
+		(property "Footprint" "Connector_PinHeader_2.54mm:PinHeader_1x05_P2.54mm_Vertical"
+			(at 176.53 107.95 0)
+			(hide yes)
+			(show_name no)
+			(do_not_autoplace no)
+			(effects
+				(font
+					(size 1.27 1.27)
+				)
+			)
+		)
+		(property "Datasheet" ""
+			(at 176.53 107.95 0)
+			(hide yes)
+			(show_name no)
+			(do_not_autoplace no)
+			(effects
+				(font
+					(size 1.27 1.27)
+				)
+			)
+		)
+		(property "Description" "Generic connector, single row, 01x05, script generated"
+			(at 176.53 107.95 0)
+			(hide yes)
+			(show_name no)
+			(do_not_autoplace no)
+			(effects
+				(font
+					(size 1.27 1.27)
+				)
+			)
+		)
+		(pin "4"
+		)
+		(pin "3"
+		)
+		(pin "2"
+		)
+		(pin "1"
+		)
+		(pin "5"
+		)
+		(instances
+			(project "eda"
+				(path "/42a0047f-f4da-41b6-a5bf-510bae675ffb"
+					(reference "MotorDrawer1")
+					(unit 1)
+				)
+			)
+		)
+	)
+	(symbol
 		(lib_id "Transistor_Array:ULN2003")
 		(at 156.21 107.95 0)
@@
 	)
 	(symbol
-		(lib_id "Connector:Conn_01x04_Pin")
-		(at 177.8 139.7 0)
-		(mirror y)
+		(lib_id "Connector:Conn_01x05_Pin")
+		(at 177.8 142.24 180)
 		(unit 1)
 		(body_style 1)
@@
 		)
 		(property "Value" ""
-			(at 177.165 134.62 0)
+			(at 179.07 140.9701 0)
 			(show_name no)
 			(do_not_autoplace no)
@@
 					(size 1.27 1.27)
 				)
+				(justify right)
 			)
 		)
-		(property "Footprint" "Connector_PinHeader_2.00mm:PinHeader_1x04_P2.00mm_Vertical"
-			(at 177.8 139.7 0)
+		(property "Footprint" "Connector_PinHeader_2.54mm:PinHeader_1x05_P2.54mm_Vertical"
+			(at 177.8 142.24 0)
 			(hide yes)
 			(show_name no)
@@
 		)
 		(property "Datasheet" ""
-			(at 177.8 139.7 0)
+			(at 177.8 142.24 0)
 			(hide yes)
 			(show_name no)
@@
 			)
 		)
-		(property "Description" "Generic connector, single row, 01x04, script generated"
-			(at 177.8 139.7 0)
+		(property "Description" "Generic connector, single row, 01x05, script generated"
+			(at 177.8 142.24 0)
 			(hide yes)
 			(show_name no)
@@
 		(pin "4"
 		)
-		(pin "1"
+		(pin "3"
 		)
 		(pin "2"
 		)
-		(pin "3"
+		(pin "1"
+		)
+		(pin "5"
 		)
 		(instances

Commit message: chore: minor changes
Parts:
- LCD1: footprint Connector_PinHeader_2.00mm:PinHeader_1x10_P2.00mm_Vertical -> Connector_PinHeader_2.54mm:PinHeader_1x10_P2.54mm_Vertical
Connections:
- net GND: now also SwitchConfig1.1 (Pin_1); no longer SwitchConfig1.2 (Pin_2)
- net SW: now also SwitchConfig1.2 (Pin_2); no longer SwitchConfig1.1 (Pin_1)
Changed lines of the file:
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@@
 	(wire
 		(pts
-			(xy 113.03 102.87) (xy 128.27 102.87)
-		)
-		(stroke
-			(width 0)
-			(type default)
-		)
-	)
-	(wire
-		(pts
 			(xy 113.03 111.76) (xy 128.27 111.76)
 		)
@@
 	(wire
 		(pts
+			(xy 113.03 102.87) (xy 128.27 102.87)
+		)
+		(stroke
+			(width 0)
+			(type default)
+		)
+	)
+	(wire
+		(pts
 			(xy 120.65 55.88) (xy 128.27 55.88)
 		)
@@
 	(symbol
 		(lib_id "Connector:Conn_01x02_Pin")
-		(at 107.95 102.87 0)
+		(at 107.95 105.41 0)
+		(mirror x)
 		(unit 1)
 		(body_style 1)
@@
 		(in_pos_files yes)
 		(dnp no)
-		(fields_autoplaced yes)
 		(property "Reference" "SwitchConfig1"
-			(at 108.585 100.33 0)
+			(at 107.95 100.33 0)
 			(show_name no)
 			(do_not_autoplace no)
@@
 		)
 		(property "Value" ""
-			(at 108.585 100.33 0)
+			(at 108.585 107.95 0)
 			(show_name no)
 			(do_not_autoplace no)
@@
 		)
 		(property "Footprint" "Connector_PinHeader_2.54mm:PinHeader_1x02_P2.54mm_Vertical"
-			(at 107.95 102.87 0)
+			(at 107.95 105.41 0)
 			(hide yes)
 			(show_name no)
@@
 		)
 		(property "Datasheet" ""
-			(at 107.95 102.87 0)
+			(at 107.95 105.41 0)
 			(hide yes)
 			(show_name no)
@@
 		)
 		(property "Description" "Generic connector, single row, 01x02, script generated"
-			(at 107.95 102.87 0)
+			(at 107.95 105.41 0)
 			(hide yes)
 			(show_name no)
@@
 			)
 		)
-		(property "Footprint" "Connector_PinHeader_2.00mm:PinHeader_1x10_P2.00mm_Vertical"
+		(property "Footprint" "Connector_PinHeader_2.54mm:PinHeader_1x10_P2.54mm_Vertical"
 			(at 107.95 83.82 0)
 			(hide yes)

Commit message: chore: bump deps
Parts:
- added Fan1, Fan2: (no value), Connector_PinHeader_2.54mm:PinHeader_1x02_P2.54mm_Vertical, symbol Connector:Conn_01x02_Pin
- added R19: 330, Resistor_SMD:R_1206_3216Metric_Pad1.30x1.75mm_HandSolder, symbol Device:R
- PowerMCU1, PowerPer1: footprint Connector_PinHeader_2.54mm:PinHeader_1x02_P2.54mm_Vertical -> Connector_Samtec_HPM_THT:Samtec_HPM-02-01-x-S_Straight_1x02_Pitch5.08mm
- R1, R10, R11, R12, R13, R14, R15, R16, R17, R18, R2, R3, R4, R5, R6, R7, R8, R9: footprint Resistor_THT:R_Axial_DIN0207_L6.3mm_D2.5mm_P7.62mm_Horizontal -> Resistor_SMD:R_1206_3216Metric_Pad1.30x1.75mm_HandSolder
Connections:
- net 3.3V: now also R19.2
- net BTN: now also R19.1
- net GND: now also Fan1.1 (Pin_1), Fan2.1 (Pin_1)
- net VCC: now also Fan1.2 (Pin_2), Fan2.2 (Pin_2)
Other:
- moved on the sheet: R15, R16, R17, R18
